Commit message: [Mod] match with avp poses

File: h1_2_description/inspire_hand/inspire_hand_left.urdf (robot description, URDF)
Before this commit: robot inspire_hand_left, 19 links, 18 joints
Joints:
- joint base_joint: origin xyz=0 0 0 rpy=-1.5707963 0 3.14159 -> xyz=0 0 0 rpy=0 -1.57 1.57

File: h1_2_description/inspire_hand/inspire_hand_right.urdf (robot description, URDF)
Before this commit: robot inspire_hand_right, 19 links, 18 joints
Joints:
- joint base_joint: origin xyz=0 0 0 rpy=-1.57079 0 3.14159 -> xyz=0 0 0 rpy=0 -1.57 1.57
